File: right.kicad_pcb (KiCad board)
At the start: 2 copper layers, 152.4 x 109.7 mm, 39 parts, among them U1 74VHC4051AFT, U2 GS8051-TR

Commit message: fix array
Routing:
- net row0: track 131.4 -> 185.4 mm, vias 1 -> 7
Changed lines of the file:
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@@
     (thickness 1.6)
     (drawings 35)
-    (tracks 112)
+    (tracks 136)
     (zones 0)
     (modules 39)
@@
   (segment (start 87.138 75.946) (end 87.138 68.215) (width 0.254) (layer F.Cu) (net 17))
   (segment (start 87.138 68.215) (end 87.122 68.199) (width 0.254) (layer F.Cu) (net 17))
-  (segment (start 87.122 68.199) (end 115.8748 68.199) (width 0.254) (layer B.Cu) (net 17))
   (segment (start 115.8748 68.199) (end 122.7582 61.3156) (width 0.254) (layer B.Cu) (net 17))
-  (segment (start 122.7582 61.3156) (end 176.7332 61.3156) (width 0.254) (layer B.Cu) (net 17))
   (segment (start 176.7332 61.3156) (end 182.372 66.9544) (width 0.254) (layer B.Cu) (net 17))
-  (segment (start 182.372 66.9544) (end 191.4652 66.9544) (width 0.254) (layer B.Cu) (net 17))
-  (segment (start 191.4652 66.9544) (end 201.4474 76.9366) (width 0.254) (layer B.Cu) (net 17))
+  (segment (start 106.188 75.946) (end 106.188 68.2084) (width 0.254) (layer F.Cu) (net 17))
+  (via (at 106.1974 68.199) (size 0.8) (drill 0.4) (layers F.Cu B.Cu) (net 17))
+  (segment (start 106.188 68.2084) (end 106.1974 68.199) (width 0.254) (layer F.Cu) (net 17))
+  (segment (start 87.122 68.199) (end 106.1974 68.199) (width 0.254) (layer B.Cu) (net 17))
+  (segment (start 106.1974 68.199) (end 115.8748 68.199) (width 0.254) (layer B.Cu) (net 17))
+  (via (at 125.2728 61.341) (size 0.8) (drill 0.4) (layers F.Cu B.Cu) (net 17))
+  (segment (start 125.238 61.3758) (end 125.2728 61.341) (width 0.254) (layer F.Cu) (net 17))
+  (segment (start 125.238 69.596) (end 125.238 61.3758) (width 0.254) (layer F.Cu) (net 17))
+  (segment (start 122.7582 61.3156) (end 125.2728 61.341) (width 0.254) (layer B.Cu) (net 17))
+  (via (at 144.3482 61.341) (size 0.8) (drill 0.4) (layers F.Cu B.Cu) (net 17))
+  (segment (start 144.288 61.4012) (end 144.3482 61.341) (width 0.254) (layer F.Cu) (net 17))
+  (segment (start 144.288 69.596) (end 144.288 61.4012) (width 0.254) (layer F.Cu) (net 17))
+  (segment (start 125.2728 61.341) (end 144.3482 61.341) (width 0.254) (layer B.Cu) (net 17))
+  (via (at 163.322 61.3156) (size 0.8) (drill 0.4) (layers F.Cu B.Cu) (net 17))
+  (segment (start 163.338 61.3316) (end 163.322 61.3156) (width 0.254) (layer F.Cu) (net 17))
+  (segment (start 163.338 69.596) (end 163.338 61.3316) (width 0.254) (layer F.Cu) (net 17))
+  (segment (start 144.3482 61.341) (end 163.322 61.3156) (width 0.254) (layer B.Cu) (net 17))
+  (segment (start 163.322 61.3156) (end 176.7332 61.3156) (width 0.254) (layer B.Cu) (net 17))
+  (via (at 182.372 66.9544) (size 0.8) (drill 0.4) (layers F.Cu B.Cu) (net 17))
+  (segment (start 182.388 74.676) (end 182.388 66.9704) (width 0.254) (layer F.Cu) (net 17))
+  (segment (start 182.388 66.9704) (end 182.372 66.9544) (width 0.254) (layer F.Cu) (net 17))
+  (segment (start 201.438 84.836) (end 201.438 76.946) (width 0.254) (layer F.Cu) (net 17))
+  (via (at 201.4474 76.9366) (size 0.8) (drill 0.4) (layers F.Cu B.Cu) (net 17))
+  (segment (start 201.438 76.946) (end 201.4474 76.9366) (width 0.254) (layer F.Cu) (net 17))
+  (segment (start 191.4144 67.0052) (end 191.3636 66.9544) (width 0.254) (layer B.Cu) (net 17))
+  (segment (start 191.4144 76.9366) (end 191.4144 67.0052) (width 0.254) (layer B.Cu) (net 17))
+  (segment (start 182.372 66.9544) (end 191.3636 66.9544) (width 0.254) (layer B.Cu) (net 17))
+  (segment (start 201.4474 76.9366) (end 191.4144 76.9366) (width 0.254) (layer B.Cu) (net 17))
   (segment (start 173.590001 122.790001) (end 176.130001 122.790001) (width 0.254) (layer B.Cu) (net 18))
   (segment (start 176.130001 122.790001) (end 187.96 134.62) (width 0.254) (layer B.Cu) (net 18))

Commit message: wip
Parts:
- added C2: 1u, Capacitor_SMD:C_0402_1005Metric, F.Cu at (134.0, 82.4)
- added C3: 0.1u, Capacitor_SMD:C_0402_1005Metric, F.Cu at (132.7, 82.5)
- added C4: 10u, Capacitor_SMD:C_0603_1608Metric, F.Cu at (148.1, 63.5)
- added C5: 22p, Capacitor_SMD:C_0402_1005Metric, F.Cu at (153.7, 101.2)
- added C6: 22p, Capacitor_SMD:C_0402_1005Metric, F.Cu at (142.5, 101.3)
- added D1: 1A, Diode_SMD:D_PowerDI-123, F.Cu at (132.6, 73.7)
- added F1: 500m, Fuse:Fuse_1210_3225Metric, F.Cu at (132.6, 76.8)
- added R10: 22, Resistor_SMD:R_0402_1005Metric, F.Cu at (154.9, 71.9)
- added R11: 5.1k, Resistor_SMD:R_0402_1005Metric, F.Cu at (153.4, 71.9)
- added R12: 5.1k, Resistor_SMD:R_0402_1005Metric, F.Cu at (152.1, 71.9)
- added R13: 10k, Resistor_SMD:R_0603_1608Metric, F.Cu at (146.1, 63.5)
- added R9: 22, Resistor_SMD:R_0402_1005Metric, F.Cu at (156.2, 71.9)
- added REF**: MountingHole_2.2mm_M2, MountingHole:MountingHole_2.2mm_M2, F.Cu at (126.8, 119.2)
- added REF**: MountingHole_2.2mm_M2, MountingHole:MountingHole_2.2mm_M2, F.Cu at (97.7, 75.9)
- added REF**: MountingHole_2.2mm_M2, MountingHole:MountingHole_2.2mm_M2, F.Cu at (135.8, 69.6)
- added REF**: MountingHole_2.2mm_M2, MountingHole:MountingHole_2.2mm_M2, F.Cu at (97.6, 133.1)
- added REF**: MountingHole_2.2mm_M2, MountingHole:MountingHole_2.2mm_M2, F.Cu at (208.7, 115.8)
- added REF**: MountingHole_2.2mm_M2, MountingHole:MountingHole_2.2mm_M2, F.Cu at (183.0, 63.4)
- added REF**: MountingHole_2.2mm_M2, MountingHole:MountingHole_2.2mm_M2, F.Cu at (112.2, 63.0)
- added REF**: MountingHole_2.2mm_M2, MountingHole:MountingHole_2.2mm_M2, F.Cu at (154.8, 107.8)
- added REF**: MountingHole_2.2mm_M2, MountingHole:MountingHole_2.2mm_M2, F.Cu at (221.1, 132.2)
- added REF**: MountingHole_2.2mm_M2, MountingHole:MountingHole_2.2mm_M2, F.Cu at (207.3, 155.7)
- added REF**: MountingHole_2.2mm_M2, MountingHole:MountingHole_2.2mm_M2, F.Cu at (162.1, 124.6)
- added S1: B3FS-1010P, base:SW_B3FS-1010P, F.Cu at (144.5, 58.4)
- added U3: ATMEGA32U4, base:ATmega32U4, F.Cu at (154.9, 82.5)
- added U4: PJ-327A, base:PJ-327A, F.Cu at (197.9, 62.5)
- added USB1: Wurth-632723300011, base:Wurth-632723300011-HandSoldering, F.Cu at (154.8, 55.8)
- added Y1: Crystal, base:Crystal_SMD_HC49-SD_HandSoldering, F.Cu at (148.4, 95.4)
- C1: footprint Resistor_SMD:R_0201_0603Metric -> Resistor_SMD:R_0402_1005Metric
- moved C1 0.25 mm to (115.8, 92.8), turned to 0 degrees
Connections:
- net +5V renamed VCC
