File: right.kicad_pcb (KiCad board)
At the start: 2 copper layers, 152.4 x 109.7 mm, 67 parts, among them U1 74VHC4051AFT, U2 GS8051-TR, U3 ATMEGA32U4, U4 PJ-327A, Y1 Crystal

Commit message: up
Parts:
- removed the REF** at (135.8, 69.6)
- removed the REF** at (154.8, 107.8)
- moved TP13 4.00 mm to (145.3, 65.6)
- moved TP14 4.00 mm to (145.3, 84.6)
- moved TP15 4.00 mm to (145.3, 103.7)
- moved Y1 1.80 mm to (148.5, 93.6)
Routing:
- net row0: track 185.4 -> 195.4 mm
- net row2: track 180.2 -> 189.8 mm
- net row1: track 179.8 -> 187.4 mm

Commit message: before autoroute
Parts:
- removed REF** (x9): MountingHole_2.2mm_M2, MountingHole:MountingHole_2.2mm_M2
- added H1: MountingHole, MountingHole:MountingHole_2.2mm_M2, F.Cu at (220.9, 132.6)
- added H2: MountingHole, MountingHole:MountingHole_2.2mm_M2, F.Cu at (97.7, 75.9)
- added H3: MountingHole, MountingHole:MountingHole_2.2mm_M2, F.Cu at (207.0, 155.6)
- added H4: MountingHole, MountingHole:MountingHole_2.2mm_M2, F.Cu at (127.1, 119.0)
- added H5: MountingHole, MountingHole:MountingHole_2.2mm_M2, F.Cu at (208.8, 116.3)
- added H6: MountingHole, MountingHole:MountingHole_2.2mm_M2, F.Cu at (97.7, 133.1)
- added H7: MountingHole, MountingHole:MountingHole_2.2mm_M2, F.Cu at (182.1, 63.1)
- added H8: MountingHole, MountingHole:MountingHole_2.2mm_M2, F.Cu at (112.0, 63.4)
- added H9: MountingHole, MountingHole:MountingHole_2.2mm_M2, F.Cu at (162.6, 120.1)
- moved USB1 2.61 mm to (157.0, 54.4)
- moved R11 1.51 mm to (151.9, 71.9)
- moved R12 1.14 mm to (153.3, 71.9)
Routing:
- net row1: track 187.4 -> 188.7 mm
- net row2: track 189.8 -> 191.0 mm

Commit message: sloppy version
Parts:
- moved U3 33.0 mm to (153.0, 115.5)
- moved Y1 31.3 mm to (137.5, 123.0), turned to 270 degrees
- moved C3 26.9 mm to (154.8, 97.7)
- moved F1 25.1 mm to (157.6, 78.4), turned to 90 degrees
- moved C2 24.7 mm to (153.4, 97.7)
- moved U1 23.1 mm to (158.0, 97.0)
- moved R7 21.2 mm to (138.8, 109.0)
- moved C1 21.2 mm to (136.0, 99.2)
- moved U2 21.2 mm to (135.0, 109.0)
- moved R8 21.2 mm to (133.7, 112.8)
- moved R5 21.2 mm to (136.3, 101.4)
- moved R6 21.2 mm to (136.3, 103.9)
- moved C5 17.6 mm to (142.8, 115.1)
- moved D1 16.0 mm to (148.6, 73.7), turned to 270 degrees
- moved C6 14.0 mm to (144.8, 115.1)
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Connections:
- U3 pad 1: Net-(U3-Pad1) -> selb
- U3 pad 10: Net-(U3-Pad10) -> col2
- U3 pad 11: Net-(U3-Pad11) -> col3
- U3 pad 18: Net-(U3-Pad18) -> scl
- U3 pad 19: Net-(U3-Pad19) -> sda
- U3 pad 28: Net-(U3-Pad28) -> col4
- U3 pad 29: Net-(U3-Pad29) -> col5
- U3 pad 30: Net-(U3-Pad30) -> col6
- U3 pad 31: Net-(U3-Pad31) -> drain
- U3 pad 32: Net-(U3-Pad32) -> inh
- U3 pad 33: Net-(U3-Pad33) -> sela
- U3 pad 41: Net-(U3-Pad41) -> read
- U3 pad 8: Net-(U3-Pad8) -> col0
- U3 pad 9: Net-(U3-Pad9) -> col1
- U4 pad 2: Net-(U4-Pad2) -> sda
- U4 pad 3: Net-(U4-Pad3) -> VCC
- U4 pad 4: Net-(U4-Pad4) -> GND
- U4 pad 5: Net-(U4-Pad5) -> scl
- U4 pad 6: Net-(U4-Pad6) -> sda
- USB1 pad 9: Net-(USB1-Pad9) -> VBUS
Routing:
- net GND: track 0.00 -> 758.8 mm, vias 0 -> 1
- net col2: track 0.00 -> 61.0 mm
- net col1: track 0.00 -> 57.2 mm
- net col0: track 0.00 -> 57.2 mm
- net col5: track 0.00 -> 38.1 mm
- net col4: track 0.00 -> 38.1 mm
- net col3: track 0.00 -> 38.1 mm
- net Net-(R9-Pad2): track 0.00 -> 26.1 mm
- net VBUS: track 0.00 -> 23.1 mm, vias 0 -> 2
- net col6: track 0.00 -> 19.0 mm
- net Net-(D1-Pad2): track 0.00 -> 11.4 mm
- net Net-(R10-Pad2): track 0.00 -> 7.27 mm
- net Net-(R12-Pad2): track 0.00 -> 7.16 mm
- net VCC: track 0.00 -> 4.46 mm
- net Net-(R11-Pad1): track 0.00 -> 1.48 mm

Commit message: minor change
Parts:
- moved C1 13.6 mm to (135.2, 112.8), turned to 270 degrees
- moved R6 12.1 mm to (133.8, 115.8), turned to 90 degrees
- moved C6 10.5 mm to (140.6, 124.8)
- moved R5 10.5 mm to (137.6, 111.8)
- moved R7 8.73 mm to (131.8, 114.2)
- moved C5 2.23 mm to (140.6, 115.4)
- moved U3 1.03 mm to (153.4, 116.4)
Changed lines of the file:
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@@
   )
   (module Resistor_SMD:R_0402_1005Metric (layer F.Cu)
-    (at 136 99.2)
+    (at 135.2 112.8 270)
     (descr "Resistor SMD 0402 (1005 Metric), square (rectangular) end terminal, IPC_7351 nominal, (Body size source: http://www.tortai-tech.com/upload/download/2011102023233369053.pdf), generated with kicad-footprint-generator")
     (tags resistor)
     (attr smd)
-    (fp_text reference C1 (at 0 -1.17) (layer F.SilkS)
-      (effects (font (size 1 1) (thickness 0.15)))
-    )
-    (fp_text value 1n (at 0 1.17) (layer F.Fab)
-      (effects (font (size 1 1) (thickness 0.15)))
-    )
-    (fp_text user %R (at 0 0) (layer F.Fab)
+    (fp_text reference C1 (at 0 -1.17 90) (layer F.SilkS)
+      (effects (font (size 1 1) (thickness 0.15)))
+    )
+    (fp_text value 1n (at 0 1.17 90) (layer F.Fab)
+      (effects (font (size 1 1) (thickness 0.15)))
+    )
+    (fp_text user %R (at 0 0 90) (layer F.Fab)
       (effects (font (size 0.25 0.25) (thickness 0.04)))
     )
@@
     (fp_line (start -0.5 -0.25) (end 0.5 -0.25) (layer F.Fab) (width 0.1))
     (fp_line (start -0.5 0.25) (end -0.5 -0.25) (layer F.Fab) (width 0.1))
-    (pad 2 smd roundrect (at 0.485 0) (size 0.59 0.64) (layers F.Cu F.Paste F.Mask) (roundrect_rratio 0.25)
-      (net 1 GND))
-    (pad 1 smd roundrect (at -0.485 0) (size 0.59 0.64) (layers F.Cu F.Paste F.Mask) (roundrect_rratio 0.25)
+    (pad 2 smd roundrect (at 0.485 0 270) (size 0.59 0.64) (layers F.Cu F.Paste F.Mask) (roundrect_rratio 0.25)
+      (net 1 GND))
+    (pad 1 smd roundrect (at -0.485 0 270) (size 0.59 0.64) (layers F.Cu F.Paste F.Mask) (roundrect_rratio 0.25)
       (net 2 row))
     (model ${KISYS3DMOD}/Resistor_SMD.3dshapes/R_0402_1005Metric.wrl
@@
   )
   (module base:ATmega32U4 (layer F.Cu)
-    (at 153 115.45)
+    (at 153.4 116.4)
     (attr smd)
     (fp_text reference U3 (at 0 9.04357) (layer F.SilkS)
@@
   )
   (module Capacitor_SMD:C_0402_1005Metric (layer F.Cu)
-    (at 144.75 115.135 270)
+    (at 140.6 124.8 270)
     (descr "Capacitor SMD 0402 (1005 Metric), square (rectangular) end terminal, IPC_7351 nominal, (Body size source: http://www.tortai-tech.com/upload/download/2011102023233369053.pdf), generated with kicad-footprint-generator")
     (tags capacitor)
@@
   )
   (module Capacitor_SMD:C_0402_1005Metric (layer F.Cu)
-    (at 142.8 115.06 270)
+    (at 140.6 115.4 270)
     (descr "Capacitor SMD 0402 (1005 Metric), square (rectangular) end terminal, IPC_7351 nominal, (Body size source: http://www.tortai-tech.com/upload/download/2011102023233369053.pdf), generated with kicad-footprint-generator")
     (tags capacitor)
@@
   )
   (module Resistor_SMD:R_1206_3216Metric (layer F.Cu)
-    (at 138.818 109.016 270)
+    (at 131.8 114.2 270)
     (descr "Resistor SMD 1206 (3216 Metric), square (rectangular) end terminal, IPC_7351 nominal, (Body size source: http://www.tortai-tech.com/upload/download/2011102023233369053.pdf), generated with kicad-footprint-generator")
     (tags resistor)
@@
   )
   (module Resistor_SMD:R_0603_1608Metric (layer F.Cu)
-    (at 136.278 103.936)
+    (at 133.8 115.8 90)
     (descr "Resistor SMD 0603 (1608 Metric), square (rectangular) end terminal, IPC_7351 nominal, (Body size source: http://www.tortai-tech.com/upload/download/2011102023233369053.pdf), generated with kicad-footprint-generator")
     (tags resistor)
     (attr smd)
-    (fp_text reference R6 (at 0 -1.43) (layer F.SilkS)
-      (effects (font (size 1 1) (thickness 0.15)))
-    )
-    (fp_text value 330 (at 0 1.43) (layer F.Fab)
+    (fp_text reference R6 (at 0 -1.43 90) (layer F.SilkS)
+      (effects (font (size 1 1) (thickness 0.15)))
+    )
+    (fp_text value 330 (at 0 1.43 90) (layer F.Fab)
       (effects (font (size 1 1) (thickness 0.15)))
     )
@@
     (fp_line (start 1.48 -0.73) (end 1.48 0.73) (layer F.CrtYd) (width 0.05))
     (fp_line (start 1.48 0.73) (end -1.48 0.73) (layer F.CrtYd) (width 0.05))
-    (fp_text user %R (at 0 0) (layer F.Fab)
+    (fp_text user %R (at 0 0 90) (layer F.Fab)
       (effects (font (size 0.4 0.4) (thickness 0.06)))
     )
-    (pad 1 smd roundrect (at -0.7875 0) (size 0.875 0.95) (layers F.Cu F.Paste F.Mask) (roundrect_rratio 0.25)
+    (pad 1 smd roundrect (at -0.7875 0 90) (size 0.875 0.95) (layers F.Cu F.Paste F.Mask) (roundrect_rratio 0.25)
       (net 2 row))
-    (pad 2 smd roundrect (at 0.7875 0) (size 0.875 0.95) (layers F.Cu F.Paste F.Mask) (roundrect_rratio 0.25)
+    (pad 2 smd roundrect (at 0.7875 0 90) (size 0.875 0.95) (layers F.Cu F.Paste F.Mask) (roundrect_rratio 0.25)
       (net 19 "Net-(R6-Pad2)"))
     (model ${KISYS3DMOD}/Resistor_SMD.3dshapes/R_0603_1608Metric.wrl
@@
   )
   (module Resistor_SMD:R_0603_1608Metric (layer F.Cu)
-    (at 136.278 101.396 180)
+    (at 137.6 111.8 180)
     (descr "Resistor SMD 0603 (1608 Metric), square (rectangular) end terminal, IPC_7351 nominal, (Body size source: http://www.tortai-tech.com/upload/download/2011102023233369053.pdf), generated with kicad-footprint-generator")
     (tags resistor)

Commit message: test
Parts:
- moved C2 24.3 mm to (140.6, 118.3)
- moved C3 23.2 mm to (144.2, 118.3)
- moved R13 10.3 mm to (154.6, 83.2)
- moved C4 1.65 mm to (153.0, 71.8), turned to 90 degrees
Routing:
- net VCC: track 4.46 -> 30.9 mm
- net GND: track 758.8 -> 768.0 mm
Changed lines of the file:
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@@
     (thickness 1.6)
     (drawings 35)
-    (tracks 360)
+    (tracks 373)
     (zones 0)
     (modules 65)
@@
   )
   (module Resistor_SMD:R_0603_1608Metric (layer F.Cu)
-    (at 151.1 73.475 270)
+    (at 154.6 83.2 270)
     (descr "Resistor SMD 0603 (1608 Metric), square (rectangular) end terminal, IPC_7351 nominal, (Body size source: http://www.tortai-tech.com/upload/download/2011102023233369053.pdf), generated with kicad-footprint-generator")
     (tags resistor)
@@
   )
   (module Capacitor_SMD:C_0603_1608Metric (layer F.Cu)
-    (at 153 73.45 270)
+    (at 153 71.8 90)
     (descr "Capacitor SMD 0603 (1608 Metric), square (rectangular) end terminal, IPC_7351 nominal, (Body size source: http://www.tortai-tech.com/upload/download/2011102023233369053.pdf), generated with kicad-footprint-generator")
     (tags capacitor)
@@
     (fp_line (start -0.8 -0.4) (end 0.8 -0.4) (layer F.Fab) (width 0.1))
     (fp_line (start -0.8 0.4) (end -0.8 -0.4) (layer F.Fab) (width 0.1))
-    (pad 2 smd roundrect (at 0.7875 0 270) (size 0.875 0.95) (layers F.Cu F.Paste F.Mask) (roundrect_rratio 0.25)
-      (net 1 GND))
-    (pad 1 smd roundrect (at -0.7875 0 270) (size 0.875 0.95) (layers F.Cu F.Paste F.Mask) (roundrect_rratio 0.25)
+    (pad 2 smd roundrect (at 0.7875 0 90) (size 0.875 0.95) (layers F.Cu F.Paste F.Mask) (roundrect_rratio 0.25)
+      (net 1 GND))
+    (pad 1 smd roundrect (at -0.7875 0 90) (size 0.875 0.95) (layers F.Cu F.Paste F.Mask) (roundrect_rratio 0.25)
       (net 23 VCC))
     (model ${KISYS3DMOD}/Capacitor_SMD.3dshapes/C_0603_1608Metric.wrl
@@
   )
   (module Capacitor_SMD:C_0402_1005Metric (layer F.Cu)
-    (at 154.8 97.715 90)
+    (at 144.2 118.315 90)
     (descr "Capacitor SMD 0402 (1005 Metric), square (rectangular) end terminal, IPC_7351 nominal, (Body size source: http://www.tortai-tech.com/upload/download/2011102023233369053.pdf), generated with kicad-footprint-generator")
     (tags capacitor)
@@
   )
   (module Capacitor_SMD:C_0402_1005Metric (layer F.Cu)
-    (at 153.4 97.715 270)
+    (at 140.6 118.315 270)
     (descr "Capacitor SMD 0402 (1005 Metric), square (rectangular) end terminal, IPC_7351 nominal, (Body size source: http://www.tortai-tech.com/upload/download/2011102023233369053.pdf), generated with kicad-footprint-generator")
     (tags capacitor)
@@
   (segment (start 183.388 80.563357) (end 183.981653 81.15701) (width 0.254) (layer B.Cu) (net 1))
   (segment (start 183.388 74.676) (end 183.388 80.563357) (width 0.254) (layer B.Cu) (net 1))
+  (segment (start 152.525 71.0125) (end 153 71.0125) (width 0.254) (layer F.Cu) (net 1))
+  (segment (start 152.055 70.5425) (end 152.525 71.0125) (width 0.254) (layer F.Cu) (net 1))
+  (segment (start 152.055 62.48) (end 152.055 70.5425) (width 0.254) (layer F.Cu) (net 1))
   (segment (start 203.438 84.836) (end 203.438 103.886) (width 0.254) (layer F.Cu) (net 3))
   (segment (start 184.388 74.676) (end 184.388 93.726) (width 0.254) (layer F.Cu) (net 4))
@@
   (segment (start 148.7375 72.6625) (end 148.6 72.8) (width 0.254) (layer F.Cu) (net 23))
   (segment (start 153 72.6625) (end 148.7375 72.6625) (width 0.254) (layer F.Cu) (net 23))
+  (segment (start 147.468999 76.004801) (end 153.876698 82.4125) (width 0.254) (layer F.Cu) (net 23))
+  (segment (start 153.876698 82.4125) (end 154.125 82.4125) (width 0.254) (layer F.Cu) (net 23))
+  (segment (start 147.468999 72.927001) (end 147.468999 76.004801) (width 0.254) (layer F.Cu) (net 23))
+  (segment (start 147.596 72.8) (end 147.468999 72.927001) (width 0.254) (layer F.Cu) (net 23))
+  (segment (start 154.125 82.4125) (end 154.6 82.4125) (width 0.254) (layer F.Cu) (net 23))
+  (segment (start 148.6 72.8) (end 147.596 72.8) (width 0.254) (layer F.Cu) (net 23))
+  (segment (start 155.725 93.296) (end 155.725 94.075) (width 0.254) (layer F.Cu) (net 23))
+  (segment (start 155.725 83.0625) (end 155.725 93.296) (width 0.254) (layer F.Cu) (net 23))
+  (segment (start 155.075 82.4125) (end 155.725 83.0625) (width 0.254) (layer F.Cu) (net 23))
+  (segment (start 154.6 82.4125) (end 155.075 82.4125) (width 0.254) (layer F.Cu) (net 23))
   (segment (start 148.6 75.954) (end 148.6 75.175) (width 0.254) (layer F.Cu) (net 26))
   (segment (start 152.446 79.8) (end 148.6 75.954) (width 0.254) (layer F.Cu) (net 26))

Commit message: wip
Parts:
- R5: moved to B.Cu
- moved Y1 38.0 mm to (174.5, 114.1)
- moved U1 33.3 mm to (139.1, 124.4), turned to 180 degrees
- moved C5 29.8 mm to (170.3, 114.1), turned to 90 degrees
- moved C6 29.2 mm to (168.9, 117.3)
- moved R5 13.8 mm to (151.3, 113.4), turned to 270 degrees
- moved C2 13.5 mm to (153.2, 122.9), turned to 0 degrees
- moved R7 12.5 mm to (143.7, 117.8)
- moved U2 10.2 mm to (140.5, 117.6)
- moved R8 7.12 mm to (138.2, 118.4), turned to 270 degrees
- moved R6 6.74 mm to (140.4, 114.3), turned to 180 degrees
- moved C3 1.62 mm to (145.8, 118.0), turned to 270 degrees
- moved U3 1.12 mm to (153.6, 115.3), turned to 90 degrees
Routing:
- net Net-(R13-Pad2): track 0.00 -> 78.1 mm, vias 0 -> 4
- net scl: track 0.00 -> 74.4 mm, vias 0 -> 4
- net sda: track 0.00 -> 73.3 mm, vias 0 -> 2
- net VCC: track 30.9 -> 99.7 mm, vias 0 -> 5
- net D-: track 0.00 -> 55.7 mm, vias 0 -> 4
- net D+: track 0.00 -> 53.8 mm, vias 0 -> 2
- net VBUS: track 23.1 -> 70.6 mm, vias 2 -> 6
- net GND: track 768.0 -> 795.9 mm, vias 1 -> 2
- net sela: track 0.00 -> 24.8 mm
- net Net-(C5-Pad1): track 0.00 -> 21.2 mm
- net inh: track 0.00 -> 19.5 mm, vias 0 -> 2
- net Net-(C6-Pad1): track 0.00 -> 17.5 mm
- net row: track 0.00 -> 10.1 mm, vias 0 -> 1
- net read: track 0.00 -> 6.72 mm
- net Net-(R7-Pad2): track 0.00 -> 6.61 mm
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
Commit message: wip
Parts:
- moved C1 5.50 mm to (140.7, 112.9), turned to 180 degrees
Routing:
- net col6: track 19.0 -> 158.1 mm, vias 0 -> 4
- net col0: track 57.2 -> 145.0 mm, vias 0 -> 2
- net row0: track 195.4 -> 275.7 mm, vias 7 -> 8
- net col5: track 38.1 -> 117.6 mm, vias 0 -> 2
- net col4: track 38.1 -> 112.6 mm, vias 0 -> 2
- net GND: track 795.9 -> 864.7 mm, vias 2 -> 5
- net col3: track 38.1 -> 106.2 mm, vias 0 -> 2
- net col1: track 57.2 -> 125.0 mm, vias 0 -> 2
- net row1: track 188.7 -> 245.3 mm, vias 7 -> 8
- net VCC: track 99.7 -> 154.4 mm, vias 5 -> 11
- net col2: track 61.0 -> 109.8 mm, vias 0 -> 2
- net row2: track 191.0 -> 233.8 mm, vias 7 -> 8
- net selb: track 0.00 -> 22.6 mm, vias 0 -> 4
- net row: track 10.1 -> 25.4 mm, vias 1 -> 2
- net row3: track 190.7 -> 199.2 mm, vias 7 -> 8
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
Commit message: sloppy version
Routing:
- net GND: track 864.7 -> 1097.5 mm, vias 5 -> 15
- net Net-(R13-Pad2): track 79.5 -> 80.5 mm
