File: right.kicad_pcb (KiCad board)
At the start: 2 copper layers, 152.4 x 109.7 mm, 65 parts, among them U1 74VHC4051AFT, U2 GS8051-TR, U3 ATMEGA32U4, U4 PJ-327A, Y1 Crystal

Commit message: add pull up
Parts:
- added R14: 5.1k, Resistor_SMD:R_0402_1005Metric, B.Cu at (194.8, 67.4)
- added R15: 5.1k, Resistor_SMD:R_0402_1005Metric, B.Cu at (194.3, 69.3)
Routing:
- net GND: track 1117.1 -> 1146.4 mm, vias 18 -> 19
- net scl: track 74.4 -> 78.8 mm
- net VCC: track 154.4 -> 158.1 mm, vias 15 -> 16
- net sda: track 73.2 -> 75.5 mm, vias 2 -> 3
- removed copper zone on B.Cu, net GND
- removed copper zone on F.Cu, net GND
Changed lines of the file:
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@@
     (thickness 1.6)
     (drawings 35)
-    (tracks 973)
+    (tracks 995)
     (zones 0)
-    (modules 65)
+    (modules 67)
     (nets 59)
   )
@@
     (add_net selb)
   )
+  (module Resistor_SMD:R_0402_1005Metric (layer B.Cu)
+    (at 194.31 69.319 90)
+    (descr "Resistor SMD 0402 (1005 Metric), square (rectangular) end terminal, IPC_7351 nominal, (Body size source: http://www.tortai-tech.com/upload/download/2011102023233369053.pdf), generated with kicad-footprint-generator")
+    (tags resistor)
+    (attr smd)
+    (fp_text reference R15 (at 0 1.17 90) (layer B.SilkS)
+      (effects (font (size 1 1) (thickness 0.15)) (justify mirror))
+    )
+    (fp_text value 5.1k (at 0 -1.17 90) (layer B.Fab)
+      (effects (font (size 1 1) (thickness 0.15)) (justify mirror))
+    )
+    (fp_text user %R (at 0 0 90) (layer B.Fab)
+      (effects (font (size 0.25 0.25) (thickness 0.04)) (justify mirror))
+    )
+    (fp_line (start 0.93 -0.47) (end -0.93 -0.47) (layer B.CrtYd) (width 0.05))
+    (fp_line (start 0.93 0.47) (end 0.93 -0.47) (layer B.CrtYd) (width 0.05))
+    (fp_line (start -0.93 0.47) (end 0.93 0.47) (layer B.CrtYd) (width 0.05))
+    (fp_line (start -0.93 -0.47) (end -0.93 0.47) (layer B.CrtYd) (width 0.05))
+    (fp_line (start 0.5 -0.25) (end -0.5 -0.25) (layer B.Fab) (width 0.1))
+    (fp_line (start 0.5 0.25) (end 0.5 -0.25) (layer B.Fab) (width 0.1))
+    (fp_line (start -0.5 0.25) (end 0.5 0.25) (layer B.Fab) (width 0.1))
+    (fp_line (start -0.5 -0.25) (end -0.5 0.25) (layer B.Fab) (width 0.1))
+    (pad 2 smd roundrect (at 0.485 0 90) (size 0.59 0.64) (layers B.Cu B.Paste B.Mask) (roundrect_rratio 0.25)
+      (net 23 VCC))
+    (pad 1 smd roundrect (at -0.485 0 90) (size 0.59 0.64) (layers B.Cu B.Paste B.Mask) (roundrect_rratio 0.25)
+      (net 58 sda))
+    (model ${KISYS3DMOD}/Resistor_SMD.3dshapes/R_0402_1005Metric.wrl
+      (at (xyz 0 0 0))
+      (scale (xyz 1 1 1))
+      (rotate (xyz 0 0 0))
+    )
+  )
+  (module Resistor_SMD:R_0402_1005Metric (layer B.Cu)
+    (at 194.795 67.437 180)
+    (descr "Resistor SMD 0402 (1005 Metric), square (rectangular) end terminal, IPC_7351 nominal, (Body size source: http://www.tortai-tech.com/upload/download/2011102023233369053.pdf), generated with kicad-footprint-generator")
+    (tags resistor)
+    (attr smd)
+    (fp_text reference R14 (at 0 1.17) (layer B.SilkS)
+      (effects (font (size 1 1) (thickness 0.15)) (justify mirror))
+    )
+    (fp_text value 5.1k (at 0 -1.17) (layer B.Fab)
+      (effects (font (size 1 1) (thickness 0.15)) (justify mirror))
+    )
+    (fp_text user %R (at 0 0) (layer B.Fab)
+      (effects (font (size 0.25 0.25) (thickness 0.04)) (justify mirror))
+    )
+    (fp_line (start 0.93 -0.47) (end -0.93 -0.47) (layer B.CrtYd) (width 0.05))
+    (fp_line (start 0.93 0.47) (end 0.93 -0.47) (layer B.CrtYd) (width 0.05))
+    (fp_line (start -0.93 0.47) (end 0.93 0.47) (layer B.CrtYd) (width 0.05))
+    (fp_line (start -0.93 -0.47) (end -0.93 0.47) (layer B.CrtYd) (width 0.05))
+    (fp_line (start 0.5 -0.25) (end -0.5 -0.25) (layer B.Fab) (width 0.1))
+    (fp_line (start 0.5 0.25) (end 0.5 -0.25) (layer B.Fab) (width 0.1))
+    (fp_line (start -0.5 0.25) (end 0.5 0.25) (layer B.Fab) (width 0.1))
+    (fp_line (start -0.5 -0.25) (end -0.5 0.25) (layer B.Fab) (width 0.1))
+    (pad 2 smd roundrect (at 0.485 0 180) (size 0.59 0.64) (layers B.Cu B.Paste B.Mask) (roundrect_rratio 0.25)
+      (net 23 VCC))
+    (pad 1 smd roundrect (at -0.485 0 180) (size 0.59 0.64) (layers B.Cu B.Paste B.Mask) (roundrect_rratio 0.25)
+      (net 57 scl))
+    (model ${KISYS3DMOD}/Resistor_SMD.3dshapes/R_0402_1005Metric.wrl
+      (at (xyz 0 0 0))
+      (scale (xyz 1 1 1))
+      (rotate (xyz 0 0 0))
+    )
+  )
   (module MountingHole:MountingHole_2.2mm_M2 (layer F.Cu)
     (at 162.56 120.142)
@@
   (segment (start 107.20699 101.85201) (end 118.919347 101.85201) (width 0.254) (layer B.Cu) (net 1))
   (segment (start 118.919347 101.85201) (end 126.238 94.533357) (width 0.254) (layer B.Cu) (net 1))
-  (segment (start 126.831653 95.12701) (end 140.694347 95.12701) (width 0.254) (layer B.Cu) (net 1))
   (segment (start 126.238 94.533357) (end 126.831653 95.12701) (width 0.254) (layer B.Cu) (net 1))
   (segment (start 140.694347 95.12701) (end 145.30699 90.514367) (width 0.254) (layer B.Cu) (net 1))
@@
   (via (at 159.258 100.965) (size 0.8) (drill 0.4) (layers F.Cu B.Cu) (net 1))
   (via (at 130.175 100.33) (size 0.8) (drill 0.4) (layers F.Cu B.Cu) (net 1))
+  (segment (start 160.595 56.696) (end 160.595 57.75) (width 0.254) (layer F.Cu) (net 1))
+  (segment (start 161.684001 55.606999) (end 160.595 56.696) (width 0.254) (layer F.Cu) (net 1))
+  (segment (start 173.843999 55.606999) (end 161.684001 55.606999) (width 0.254) (layer F.Cu) (net 1))
+  (segment (start 178.435 60.198) (end 173.843999 55.606999) (width 0.254) (layer F.Cu) (net 1))
+  (segment (start 130.175 96.27402) (end 129.02799 95.12701) (width 0.254) (layer F.Cu) (net 1))
+  (segment (start 130.175 100.33) (end 130.175 96.27402) (width 0.254) (layer F.Cu) (net 1))
+  (via (at 129.02799 95.12701) (size 0.8) (drill 0.4) (layers F.Cu B.Cu) (net 1))
+  (segment (start 126.831653 95.12701) (end 129.02799 95.12701) (width 0.254) (layer B.Cu) (net 1))
+  (segment (start 129.02799 95.12701) (end 140.694347 95.12701) (width 0.254) (layer B.Cu) (net 1))
+  (segment (start 160.800999 100.565001) (end 161.29 100.076) (width 0.254) (layer B.Cu) (net 1))
+  (segment (start 159.657999 100.565001) (end 160.800999 100.565001) (width 0.254) (layer B.Cu) (net 1))
+  (segment (start 159.258 100.965) (end 159.657999 100.565001) (width 0.254) (layer B.Cu) (net 1))
   (via (at 142.56 114.25) (size 0.8) (drill 0.4) (layers F.Cu B.Cu) (net 2))
   (segment (start 151.27 114.1975) (end 142.6125 114.1975) (width 0.254) (layer B.Cu) (net 2))
@@
   (segment (start 169.6615 75.8085) (end 179.5675 65.9025) (width 0.254) (layer B.Cu) (net 23))
   (segment (start 182.394057 65.255943) (end 189.252057 65.255943) (width 0.254) (layer B.Cu) (net 23))
+  (via (at 194.31 66.421) (size 0.8) (drill 0.4) (layers F.Cu B.Cu) (net 23))
+  (segment (start 194.31 67.437) (end 194.31 66.421) (width 0.254) (layer B.Cu) (net 23))
+  (segment (start 194.31 65.14) (end 194.366 65.084) (width 0.254) (layer F.Cu) (net 23))
+  (segment (start 194.31 66.421) (end 194.31 65.14) (width 0.254) (layer F.Cu) (net 23))
+  (segment (start 194.31 67.437) (end 194.31 68.834) (width 0.254) (layer B.Cu) (net 23))
   (segment (start 174.46 112.3915) (end 174.46 108.2) (width 0.254) (layer F.Cu) (net 24))
   (segment (start 171.5415 115.31) (end 174.46 112.3915) (width 0.254) (layer F.Cu) (net 24))
@@
   (segment (start 168.0174 114.5226) (end 172.08 110.46) (width 0.254) (layer F.Cu) (net 57))
   (segment (start 159.3804 114.5226) (end 168.0174 114.5226) (width 0.254) (layer F.Cu) (net 57))
+  (segment (start 199.110998 67.437) (end 199.484999 67.811001) (width 0.254) (layer B.Cu) (net 57))
+  (segment (start 195.28 67.437) (end 199.110998 67.437) (width 0.254) (layer B.Cu) (net 57))
   (segment (start 194.366 73.088) (end 194.366 72.084) (width 0.254) (layer F.Cu) (net 58))
   (segment (start 195.062 73.784) (end 194.366 73.088) (width 0.254) (layer F.Cu) (net 58))
@@
   (segment (start 167.8002 113.7098) (end 171.32 110.19) (width 0.254) (layer F.Cu) (net 58))
   (segment (start 171.32 95.15) (end 171.302059 95.132059) (width 0.254) (layer F.Cu) (net 58))
-  (zone (net 1) (net_name GND) (layer B.Cu) (hatch edge 0.508)
-    (connect_pads (clearance 0.508))
-    (min_thickness 0.254)
-    (fill yes (arc_segments 32) (thermal_gap 0.508) (thermal_bridge_width 0.508))
-    (polygon
-      (pts
-        (xy 254.635 172.593) (xy 58.039 166.37) (xy 63.5 47.117) (xy 63.627 47.117) (xy 251.333 39.37)
-      )
-    )
-  )
+  (via (at 194.31 70.612) (size 0.8) (drill 0.4) (layers F.Cu B.Cu) (net 58))
+  (segment (start 194.31 69.804) (end 194.31 70.612) (width 0.254) (layer B.Cu) (net 58))
+  (segment (start 194.31 72.028) (end 194.366 72.084) (width 0.254) (layer F.Cu) (net 58))
+  (segment (start 194.31 70.612) (end 194.31 72.028) (width 0.254) (layer F.Cu) (net 58))
   (zone (net 0) (net_name "") (layer F.Cu) (hatch edge 0.508)
     (connect_pads (clearance 0.508))
@@
       )
     )
-  )
-  (zone (net 1) (net_name GND) (layer F.Cu) (hatch edge 0.508)
-    (connect_pads (clearance 0.508))
-    (min_thickness 0.254)
-    (fill yes (arc_segments 32) (thermal_gap 0.508) (thermal_bridge_width 0.508))
-    (polygon
-      (pts
-        (xy 255.27 172.593) (xy 58.039 166.497) (xy 64.135 46.99) (xy 251.46 39.37)
-      )
-    )
-  )
-  (zone (net 1) (net_name GND) (layer B.Cu) (hatch edge 0.508)
-    (connect_pads (clearance 0.508))
-    (min_thickness 0.254)
-    (fill yes (arc_segments 32) (thermal_gap 0.508) (thermal_bridge_width 0.508))
-    (polygon
-      (pts
-        (xy 192.278 74.295) (xy 132.207 50.546) (xy 199.136 47.498)
-      )
-    )
-  )
-  (zone (net 1) (net_name GND) (layer F.Cu) (hatch edge 0.508)
-    (connect_pads (clearance 0.508))
-    (min_thickness 0.254)
-    (fill yes (arc_segments 32) (thermal_gap 0.508) (thermal_bridge_width 0.508))
-    (polygon
-      (pts
-        (xy 169.672 103.632) (xy 155.448 110.998) (xy 153.289 67.564) (xy 167.894 63.754)
-      )
-    )
-  )
-  (zone (net 1) (net_name GND) (layer F.Cu) (hatch edge 0.508)
-    (connect_pads (clearance 0.508))
-    (min_thickness 0.254)
-    (fill yes (arc_segments 32) (thermal_gap 0.508) (thermal_bridge_width 0.508))
-    (polygon
-      (pts
-        (xy 138.303 108.585) (xy 122.936 114.173) (xy 124.206 92.202) (xy 138.303 76.581)
-      )
-    )

Commit message: fill
Routing:
- added copper zone on B.Cu, net GND
- added copper zone on F.Cu, net GND
Changed lines of the file:
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@@
+    )
+  )
+  (zone (net 1) (net_name GND) (layer F.Cu) (hatch edge 0.508)
+    (connect_pads (clearance 0.508))
+    (min_thickness 0.254)
+    (fill yes (arc_segments 32) (thermal_gap 0.508) (thermal_bridge_width 0.508))
+    (polygon
+      (pts
+        (xy 247.142 41.656) (xy 241.427 186.69) (xy 40.132 173.863) (xy 46.609 37.338)
+      )
+    )
+  )
+  (zone (net 1) (net_name GND) (layer B.Cu) (hatch edge 0.508)
+    (connect_pads (clearance 0.508))
+    (min_thickness 0.254)
+    (fill yes (arc_segments 32) (thermal_gap 0.508) (thermal_bridge_width 0.508))
+    (polygon
+      (pts
+        (xy 248.539 41.021) (xy 243.713 187.706) (xy 38.481 174.244) (xy 47.498 38.227)
+      )
     )
   )

Commit message: sloppy fixhh
Parts:
- moved R11 6.01 mm to (151.8, 69.5), turned to 180 degrees
- moved C4 1.75 mm to (151.3, 71.6)
- moved R10 1.40 mm to (155.4, 73.1)
Routing:
- net Net-(R9-Pad2): track 26.1 -> 38.8 mm, vias 0 -> 2
- net GND: track 1146.4 -> 1140.3 mm
- net Net-(R11-Pad1): track 1.48 -> 7.47 mm
- net VBUS: track 73.2 -> 76.3 mm
- net Net-(R10-Pad2): track 7.27 -> 9.66 mm, vias 0 -> 2
- net VCC: track 158.1 -> 156.7 mm
- net D-: track 55.7 -> 55.0 mm

Commit message: fix jack
Connections:
- U4 pad 4: GND -> VCC
- U4 pad 6: sda -> GND
Routing:
- net GND: track 1140.3 -> 1129.0 mm
- net VCC: track 156.7 -> 164.1 mm
- net sda: track 75.5 -> 68.2 mm
