File: left.kicad_pcb (KiCad board)
At the start: 2 copper layers, 152.4 x 109.7 mm, 65 parts, among them U1 74VHC4051AFT, U2 GS8051-TR, U3 ATMEGA32U4, U4 PJ-327A, Y1 Crystal

Commit message: filled
Routing:
- net GND: track 1120.4 -> 1145.2 mm, vias 16 -> 18
- added copper zone on B.Cu, net GND
- added copper zone on F.Cu, net GND

Commit message: more and more
Routing:
- net GND: track 1145.2 -> 1157.0 mm, vias 18 -> 23
Changed lines of the file:
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@@
     (thickness 1.6)
     (drawings 35)
-    (tracks 1095)
+    (tracks 1104)
     (zones 0)
     (modules 65)
@@
   (segment (start 178.213 119.857) (end 178.627 119.443) (width 0.254) (layer F.Cu) (net 1))
   (segment (start 178.627 119.443) (end 179.259882 119.443) (width 0.254) (layer F.Cu) (net 1))
-  (via (at 181.183 127.132) (size 0.8) (drill 0.4) (layers F.Cu B.Cu) (net 1))
+  (via (at 181.183 126.746) (size 0.8) (drill 0.4) (layers F.Cu B.Cu) (net 1))
   (segment (start 179.259882 119.443) (end 181.183 121.366118) (width 0.254) (layer F.Cu) (net 1))
   (segment (start 181.183 121.366118) (end 181.183 127.132) (width 0.254) (layer F.Cu) (net 1))
@@
   (segment (start 152.52699 69.84999) (end 143.804373 69.84999) (width 0.254) (layer B.Cu) (net 1))
   (segment (start 154.350367 69.84999) (end 152.52699 69.84999) (width 0.254) (layer B.Cu) (net 1))
+  (via (at 181.991 129.921) (size 0.8) (drill 0.4) (layers F.Cu B.Cu) (net 1))
+  (via (at 121.031 62.357) (size 0.8) (drill 0.4) (layers F.Cu B.Cu) (net 1))
+  (segment (start 174.031347 90.35699) (end 170.88201 90.35699) (width 0.254) (layer B.Cu) (net 1))
+  (segment (start 174.625 96.838) (end 174.625 90.950643) (width 0.254) (layer B.Cu) (net 1))
+  (segment (start 174.625 90.950643) (end 174.031347 90.35699) (width 0.254) (layer B.Cu) (net 1))
+  (segment (start 170.88201 90.35699) (end 169.545 91.694) (width 0.254) (layer B.Cu) (net 1))
+  (via (at 168.783 92.583) (size 0.8) (drill 0.4) (layers F.Cu B.Cu) (net 1))
+  (via (at 167.767 83.058) (size 0.8) (drill 0.4) (layers F.Cu B.Cu) (net 1))
+  (via (at 190.5 93.472) (size 0.8) (drill 0.4) (layers F.Cu B.Cu) (net 1))
   (via (at 177.353 107.392) (size 0.8) (drill 0.4) (layers F.Cu B.Cu) (net 2))
   (segment (start 168.643 107.3395) (end 177.3005 107.3395) (width 0.254) (layer B.Cu) (net 2))
@@
       )
     )
+  )
+  (zone (net 1) (net_name GND) (layer F.Cu) (hatch edge 0.508)
+    (connect_pads (clearance 0.508))
+    (min_thickness 0.254)
+    (fill yes (arc_segments 32) (thermal_gap 0.508) (thermal_bridge_width 0.508))
+    (polygon
+      (pts
+        (xy 137.795 82.677) (xy 111.633 77.089) (xy 113.03 52.959) (xy 139.7 50.419)
+      )
+    )
+  )
+  (zone (net 1) (net_name GND) (layer B.Cu) (hatch edge 0.508)
+    (connect_pads (clearance 0.508))
+    (min_thickness 0.254)
+    (fill yes (arc_segments 32) (thermal_gap 0.508) (thermal_bridge_width 0.508))
+    (polygon
+      (pts
+        (xy 223.266 105.156) (xy 124.968 117.856) (xy 116.078 77.089) (xy 210.058 70.104)
+      )
+    )
+  )
+  (zone (net 1) (net_name GND) (layer F.Cu) (hatch edge 0.508)
+    (connect_pads (clearance 0.508))
+    (min_thickness 0.254)
+    (fill yes (arc_segments 32) (thermal_gap 0.508) (thermal_bridge_width 0.508))
+    (polygon
+      (pts
+        (xy 210.947 172.974) (xy 140.208 169.418) (xy 140.208 34.163) (xy 215.011 28.067)
+      )
+    )
