File: left.kicad_pcb (KiCad board)
At the start: 2 copper layers, 152.4 x 109.7 mm, 65 parts, among them U1 74VHC4051AFT, U2 GS8051-TR, U3 ATMEGA32U4, U4 PJ-327A, Y1 Crystal

Commit message: add pull up
Parts:
- added R14: 5.1k, Resistor_SMD:R_0402_1005Metric, B.Cu at (123.1, 62.5)
- added R15: 5.1k, Resistor_SMD:R_0402_1005Metric, B.Cu at (118.9, 61.5)
Routing:
- net GND: track 1157.0 -> 1175.9 mm, vias 23 -> 24
- net VCC: track 174.2 -> 177.9 mm, vias 15 -> 17
- net sda: track 75.3 -> 78.7 mm, vias 2 -> 3
- net scl: track 70.4 -> 73.8 mm, vias 2 -> 3
- removed copper zone on B.Cu, net GND
- removed copper zone on F.Cu, net GND

Commit message: fill
Routing:
- added copper zone on B.Cu, net GND
- added copper zone on F.Cu, net GND
Changed lines of the file:
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@@
+    )
+  )
+  (zone (net 1) (net_name GND) (layer F.Cu) (hatch edge 0.508)
+    (connect_pads (clearance 0.508))
+    (min_thickness 0.254)
+    (fill yes (arc_segments 32) (thermal_gap 0.508) (thermal_bridge_width 0.508))
+    (polygon
+      (pts
+        (xy 269.494 37.338) (xy 272.034 172.593) (xy 77.597 169.164) (xy 86.614 37.211)
+      )
+    )
+  )
+  (zone (net 1) (net_name GND) (layer B.Cu) (hatch edge 0.508)
+    (connect_pads (clearance 0.508))
+    (min_thickness 0.254)
+    (fill yes (arc_segments 32) (thermal_gap 0.508) (thermal_bridge_width 0.508))
+    (polygon
+      (pts
+        (xy 273.685 172.72) (xy 77.978 169.799) (xy 86.487 37.846) (xy 270.637 37.084)
+      )
     )
   )

Commit message: sloppy fixhh
Parts:
- moved R9 2.55 mm to (163.7, 67.2)
- moved R11 2.28 mm to (166.4, 62.9)
Routing:
- net Net-(R9-Pad2): track 23.0 -> 29.1 mm, vias 0 -> 2
- net VBUS: track 62.7 -> 67.7 mm
- net Net-(R11-Pad1): track 1.02 -> 6.00 mm
- net GND: track 1175.9 -> 1178.2 mm, vias 24 -> 25
- net D+: track 44.9 -> 42.7 mm

Commit message: fix jack
Connections:
- U4 pad 4: GND -> VCC
- U4 pad 6: sda -> GND
Routing:
- net sda: track 78.7 -> 86.1 mm
- net GND: track 1178.2 -> 1181.6 mm
- net VCC: track 177.9 -> 180.4 mm
